Commit message: Atualizado - xacro

File: robot_description/urdf/v2/base.xacro (robot description, xacro)
@@ -2,5 +2,5 @@
 <robot name="robot" xmlns:xacro="http://www.ros.org/wiki/xacro">
     <xacro:include filename="$(find robot_description)/urdf/v2/caster_wheel.xacro" />
-    <link name="base_footprint"/>
+    <!-- <link name="base_footprint"/> -->
     <!-- ==== BASE LINK ==== -->
     <link name="base_link">
@@ -26,4 +26,5 @@
         </inertial>
     </link>
+<!--
     <joint name="base_joint" type="fixed">
         <parent link="base_footprint"/>
@@ -31,4 +32,4 @@
         <origin xyz="0.0 0.0 ${ground_distance}" rpy="0.0 0.0 0.0"/>
         <axis xyz="0.0 0.0 0.0" />
-    </joint>
+    </joint> -->
 </robot>

Commit message: Atualizado - xacro

File: robot_description/urdf/v2/base.xacro (robot description, xacro)
@@ -2,5 +2,6 @@
 <robot name="robot" xmlns:xacro="http://www.ros.org/wiki/xacro">
     <xacro:include filename="$(find robot_description)/urdf/v2/caster_wheel.xacro" />
-    <!-- <link name="base_footprint"/> -->
+    <xacro:property name="ground_distance" value="0.05" />
+    <link name="base_footprint"/>
     <!-- ==== BASE LINK ==== -->
     <link name="base_link">
@@ -26,5 +27,4 @@
         </inertial>
     </link>
-<!--
     <joint name="base_joint" type="fixed">
         <parent link="base_footprint"/>
@@ -32,4 +32,4 @@
         <origin xyz="0.0 0.0 ${ground_distance}" rpy="0.0 0.0 0.0"/>
         <axis xyz="0.0 0.0 0.0" />
-    </joint> -->
+    </joint>
 </robot>

Commit message: Atualizado - xacro

File: robot_description/urdf/v2/base.xacro (robot description, xacro)
@@ -2,5 +2,4 @@
 <robot name="robot" xmlns:xacro="http://www.ros.org/wiki/xacro">
     <xacro:include filename="$(find robot_description)/urdf/v2/caster_wheel.xacro" />
-    <xacro:property name="ground_distance" value="0.05" />
     <link name="base_footprint"/>
     <!-- ==== BASE LINK ==== -->
@@ -30,5 +29,5 @@
         <parent link="base_footprint"/>
         <child link="base_link"/>
-        <origin xyz="0.0 0.0 ${ground_distance}" rpy="0.0 0.0 0.0"/>
+        <origin xyz="0.0 0.0 0.05" rpy="0.0 0.0 0.0"/>
         <axis xyz="0.0 0.0 0.0" />
     </joint>
